File: headset/doc/pcb/HeadsetR2.sch (EAGLE design)
At the start: 54 parts, among them U1 STM32F405RGT6, U2 MAX17043, U3 MCP73831, U4 MIC5216, U5 MIC5216, U6 MIC5219 3.3V, U7 XBEE, U8 STEVAL-MKI108V2, Y1 8MHz

Commit message: Update headset schematic revision 2 (again), almost ready for route
Connections:
- net !CS!: now also U1.PA15/JTDI(5T); no longer U1.PB12(5T)
- net MISO: now also U1.PC11(5T); no longer U1.PB14/SPI2_MISO(5T)
- net MOSI: now also U1.PC12(5T); no longer U1.PB15/SPI2_MOSI(5T)
- net SCK: now also U1.PC10(5T); no longer U1.PB13/SPI2_SCK(5T)
- net X_RX: now also U1.PA2/ADC123_IN2(5T); no longer U1.PA9/TIM1_CH2/USART1_TX(5T)
- net X_TX: now also U1.PA3/ADC123_IN3(5T); no longer U1.PA10/TIM1_CH3/USART1_RX(5T)
Other:
- note added: "9 DOF IMU"
Changed lines of the file:
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@@
 <text x="7.62" y="76.2" size="1.778" layer="97">Place near MCU</text>
 <text x="7.62" y="170.18" size="1.778" layer="97">Place near MCU</text>
-<text x="142.24" y="109.22" size="1.778" layer="97" rot="R90">Raspberry PI</text>
+<text x="142.24" y="76.2" size="1.778" layer="97" rot="R90">Raspberry PI</text>
 <text x="142.24" y="129.54" size="1.778" layer="97" rot="R90">IMU</text>
 <text x="142.24" y="144.78" size="1.778" layer="97" rot="R90">Debug</text>
 <text x="142.24" y="96.52" size="1.778" layer="97" rot="R90">GPS</text>
 <text x="30.48" y="81.28" size="1.778" layer="97" rot="R90">Radio</text>
+<text x="236.22" y="142.24" size="1.778" layer="97" rot="R90">9 DOF
+IMU</text>
 </plain>
 <instances>
@@
 </segment>
 <segment>
-<pinref part="U1" gate="G$1" pin="PA10/TIM1_CH3/USART1_RX(5T)"/>
-<wire x1="43.18" y1="81.28" x2="33.02" y2="81.28" width="0.1524" layer="91"/>
-<label x="33.02" y="81.28" size="1.778" layer="95"/>
+<pinref part="U1" gate="G$1" pin="PA3/ADC123_IN3(5T)"/>
+<wire x1="33.02" y1="99.06" x2="43.18" y2="99.06" width="0.1524" layer="91"/>
+<label x="33.02" y="99.06" size="1.778" layer="95"/>
 </segment>
 </net>
@@
 </segment>
 <segment>
-<pinref part="U1" gate="G$1" pin="PA9/TIM1_CH2/USART1_TX(5T)"/>
-<wire x1="43.18" y1="83.82" x2="33.02" y2="83.82" width="0.1524" layer="91"/>
-<label x="33.02" y="83.82" size="1.778" layer="95"/>
+<pinref part="U1" gate="G$1" pin="PA2/ADC123_IN2(5T)"/>
+<wire x1="33.02" y1="101.6" x2="43.18" y2="101.6" width="0.1524" layer="91"/>
+<label x="33.02" y="101.6" size="1.778" layer="95"/>
 </segment>
 </net>
@@
 <net name="!CS!" class="0">
 <segment>
-<pinref part="U1" gate="G$1" pin="PB12(5T)"/>
-<wire x1="139.7" y1="127" x2="129.54" y2="127" width="0.1524" layer="91"/>
-<label x="132.08" y="127" size="1.778" layer="95"/>
-</segment>
-<segment>
 <pinref part="JP6" gate="G$1" pin="2"/>
 <wire x1="233.68" y1="119.38" x2="228.6" y2="119.38" width="0.1524" layer="91"/>
@@
 <label x="248.92" y="40.64" size="1.778" layer="95"/>
 </segment>
+<segment>
+<pinref part="U1" gate="G$1" pin="PA15/JTDI(5T)"/>
+<wire x1="43.18" y1="68.58" x2="33.02" y2="68.58" width="0.1524" layer="91"/>
+<label x="33.02" y="68.58" size="1.778" layer="95"/>
+</segment>
 </net>
 <net name="SCK" class="0">
-<segment>
-<pinref part="U1" gate="G$1" pin="PB13/SPI2_SCK(5T)"/>
-<wire x1="139.7" y1="124.46" x2="129.54" y2="124.46" width="0.1524" layer="91"/>
-<label x="132.08" y="124.46" size="1.778" layer="95"/>
-</segment>
 <segment>
 <pinref part="JP6" gate="G$1" pin="5"/>
@@
 <label x="220.98" y="40.64" size="1.778" layer="95"/>
 </segment>
+<segment>
+<pinref part="U1" gate="G$1" pin="PC10(5T)"/>
+<wire x1="139.7" y1="88.9" x2="129.54" y2="88.9" width="0.1524" layer="91"/>
+<label x="132.08" y="88.9" size="1.778" layer="95"/>
+</segment>
 </net>
 <net name="MISO" class="0">
-<segment>
-<pinref part="U1" gate="G$1" pin="PB14/SPI2_MISO(5T)"/>
-<wire x1="139.7" y1="121.92" x2="129.54" y2="121.92" width="0.1524" layer="91"/>
-<label x="132.08" y="121.92" size="1.778" layer="95"/>
-</segment>
 <segment>
 <pinref part="JP6" gate="G$1" pin="3"/>
@@
 <label x="220.98" y="43.18" size="1.778" layer="95"/>
 </segment>
+<segment>
+<pinref part="U1" gate="G$1" pin="PC11(5T)"/>
+<wire x1="139.7" y1="86.36" x2="129.54" y2="86.36" width="0.1524" layer="91"/>
+<label x="132.08" y="86.36" size="1.778" layer="95"/>
+</segment>
 </net>
 <net name="MOSI" class="0">
-<segment>
-<pinref part="U1" gate="G$1" pin="PB15/SPI2_MOSI(5T)"/>
-<wire x1="139.7" y1="119.38" x2="129.54" y2="119.38" width="0.1524" layer="91"/>
-<label x="132.08" y="119.38" size="1.778" layer="95"/>
-</segment>
 <segment>
 <pinref part="JP6" gate="G$1" pin="4"/>
@@
 <label x="220.98" y="45.72" size="1.778" layer="95"/>
 </segment>
-</net>
+<segment>
+<pinref part="U1" gate="G$1" pin="PC12(5T)"/>
+<wire x1="139.7" y1="83.82" x2="129.54" y2="83.82" width="0.1524" layer="91"/>
+<label x="132.08" y="83.82" size="1.778" layer="95"/>
+</segment>
+</net>

Commit message: Update schematic revision 2 to fix the issues described in lab notebook
Parts:
- added D3: LED, SparkFun-LED:LED-RED1206
- added R10: 10K, ECE477:RES1206
- added R11: 470, ECE477:RES1206
- C22, C23, C24: device ECE477:CAP_POLVISHAY_D -> SparkFun-Passives:CAP_POLD
- JP2: value SWD -> SPARE; device SparkFun-Connectors:M06SIP -> SparkFun-Connectors:M03PTH
- JP6: device SparkFun-Connectors:M06SIP -> SparkFun-Connectors:M03PTH
Connections:
- removed net AGND: C19.2, U1.VSSA, U6.GND, U8.13
- new net LED: D3.A, U1.PC13(5T)
- new net LED_LED: D3.C, R11.2
- new net S_RX: JP2.3, R10.1, U1.PA10/TIM1_CH3/USART1_RX(5T)
- new net S_TX: JP2.1, U1.PA9/TIM1_CH2/USART1_TX(5T)
- net !CS!: no longer JP6.2
- net !RST!: no longer JP2.5
- net 5V: now also JP6.3; no longer JP6.6
- net GND: now also C19.2, JP2.2, R11.1, U1.PB2/BOOT1(5T), U1.VSSA, U6.GND, U8.13; no longer JP2.3
- net MISO: no longer JP6.3
- net MOSI: no longer JP6.4
- net SCK: no longer JP6.5
- net SWCLK: no longer JP2.2
- net SWDIO: no longer JP2.4
- net SWO: no longer JP2.6
- net V_MCU: now also R10.2, U1.PB5(5T); no longer JP2.1
Other:
- note removed: "DO NOT STUFF JP2"
