File: headset/doc/pcb/HeadsetCCup.brd (EAGLE design)
At the start: 55.8 x 50.9 mm, 41 parts, among them U1 STM32F405RGT6, U4 MIC5219, U6 MIC5219 3.3V, U8 STEVAL-MKI108V2, Y1 8MHz

Commit message: Add the latest version of Cornell Cup PCBs to repository
Parts:
- C14, C15: value 22p -> 39p
- moved C13 2.62 mm to (12.7, 23.5)
- moved C15 0.64 mm to (3.81, 27.3)
- moved C14 0.63 mm to (3.81, 33.7)
- moved C23 0.63 mm to (50.8, 41.3)
- moved C24 0.63 mm to (43.2, 41.3)
Routing:
- net V_ADC: track 44.0 -> 45.1 mm
Other:
- board text added: "Cornell Cup 2/19/14 Augmented Reality R6"
