File: headset/doc/pcb/HeadsetCCup.sch (EAGLE design)
At the start: 41 parts, among them U1 STM32F405RGT6, U4 MIC5219, U6 MIC5219 3.3V, U8 STEVAL-MKI108V2, Y1 8MHz

Commit message: Add the latest version of Cornell Cup PCBs to repository
Parts:
- C14, C15: value 22p -> 39p
Changed lines of the file:
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@@
 <part name="GND6" library="supply1" deviceset="GND" device=""/>
 <part name="Y1" library="SparkFun-FreqCtrl" deviceset="CRYSTAL" device="HC49US" value="8MHz"/>
-<part name="C14" library="ECE477" deviceset="CAP" device="1206" value="22p"/>
-<part name="C15" library="ECE477" deviceset="CAP" device="1206" value="22p"/>
+<part name="C14" library="ECE477" deviceset="CAP" device="1206" value="39p"/>
+<part name="C15" library="ECE477" deviceset="CAP" device="1206" value="39p"/>
 <part name="GND7" library="supply1" deviceset="GND" device=""/>
 <part name="R2" library="ECE477" deviceset="RES" device="1206" value="10k"/>
